Commit message: fix viz axis

File: models/model.urdf (robot description, URDF)
Before this commit: robot cyberarm, 5 links, 4 joints
Joints:
- joint arm1_to_arm2_joint: axis 1 0 0 -> -1 0 0
- joint arm2_to_arm3_joint: axis -1 0 0 -> 1 0 0
- joint arm3_to_end_effector_joint: axis 1 0 0 -> -1 0 0
- joint base_to_arm1_joint: axis 0 0 1 -> 0 0 -1
