Commit message: fix model url

File: cyber_arm/models/model.urdf (robot description, URDF)
Before this commit: robot cyberarm, 5 links, 4 joints
Links:
- link arm1_link: geometry visual mesh filename=package://cyber_arm/models/meshes/Joint1.dae
- link arm2_link: geometry visual mesh filename=package://cyber_arm/models/meshes/JointArm.dae
- link arm3_link: geometry visual mesh filename=package://cyber_arm/models/meshes/JointArm.dae
- link base_link: geometry visual mesh filename=package://cyber_arm/models/meshes/Base.dae
- link end_effector_link: geometry visual mesh filename=package://cyber_arm/models/meshes/EndEffector.dae

Commit message: add camera link

File: cyber_arm/models/model.urdf (robot description, URDF)
Before this commit: robot cyberarm, 5 links, 4 joints
Links:
- added link camera_link
Joints:
- added joint ee_to_camera: type fixed, parent end_effector_link, child camera_link, origin xyz=-0.056 0 0.10095 rpy=0 0 0

Commit message: fix camera coord convention

File: cyber_arm/models/model.urdf (robot description, URDF)
Before this commit: robot cyberarm, 6 links, 5 joints
Joints:
- joint ee_to_camera: origin xyz=-0.056 0 0.10095 rpy=0 0 0 -> xyz=-0.056 0 0.10095 rpy=0 -1.5708 1.5708

Commit message: move camera transform to a static publisher

File: cyber_arm/models/model.urdf (robot description, URDF)
Before this commit: robot cyberarm, 6 links, 5 joints
Links:
- removed link camera_link
Joints:
- removed joint ee_to_camera
